Commit message: Ladies and gentlemen, we got em

File: src/kuka/urdf/kr120r2500pro.xacro (robot description, xacro)
@@ -2,5 +2,5 @@
 <!--Generates a urdf from the macro in kr120r2500pro_macro.xacro -->
 <robot name="kuka_kr120r2500pro" xmlns:xacro="http://wiki.ros.org/xacro">
-    <xacro:include filename="$(find kuka_kr120_support)/urdf/kr120r2500pro_macro.xacro" />
+    <xacro:include filename="$(find kuka)/urdf/kr120r2500pro_macro.xacro" />
     <xacro:kuka_kr120r2500pro prefix=""/>
 </robot>

File: src/kuka/urdf/kr120r2500pro_macro.xacro (robot description, xacro)
@@ -13,11 +13,11 @@
         <origin xyz="0 0 0" rpy="0 0 0"/>
         <geometry>
-          <mesh filename="package://kuka_kr120_support/meshes/kr120r2500pro/visual/base_link.dae" />
-        </geometry>
-      </visual>
-      <collision>
-        <origin xyz="0 0 0" rpy="0 0 0"/>
-        <geometry>
-          <mesh filename="package://kuka_kr120_support/meshes/kr120r2500pro/collision/base_link.stl" />
+          <mesh filename="package://kuka/meshes/kr120r2500pro/visual/base_link.dae" />
+        </geometry>
+      </visual>
+      <collision>
+        <origin xyz="0 0 0" rpy="0 0 0"/>
+        <geometry>
+          <mesh filename="package://kuka/meshes/kr120r2500pro/collision/base_link.stl" />
         </geometry>
       </collision>
@@ -33,11 +33,11 @@
         <origin xyz="0 0 0" rpy="0 0 0"/>
         <geometry>
-          <mesh filename="package://kuka_kr120_support/meshes/kr120r2500pro/visual/link_1.dae" />
-        </geometry>
-      </visual>
-      <collision>
-        <origin xyz="0 0 0" rpy="0 0 0"/>
-        <geometry>
-          <mesh filename="package://kuka_kr120_support/meshes/kr120r2500pro/collision/link_1.stl" />
+          <mesh filename="package://kuka/meshes/kr120r2500pro/visual/link_1.dae" />
+        </geometry>
+      </visual>
+      <collision>
+        <origin xyz="0 0 0" rpy="0 0 0"/>
+        <geometry>
+          <mesh filename="package://kuka/meshes/kr120r2500pro/collision/link_1.stl" />
         </geometry>
       </collision>
@@ -53,11 +53,11 @@
         <origin xyz="0 0 0" rpy="0 0 0"/>
         <geometry>
-          <mesh filename="package://kuka_kr120_support/meshes/kr120r2500pro/visual/link_2.dae"/>
-        </geometry>
-      </visual>
-      <collision>
-        <origin xyz="0 0 0" rpy="0 0 0"/>
-        <geometry>
-          <mesh filename="package://kuka_kr120_support/meshes/kr120r2500pro/collision/link_2.stl" />
+          <mesh filename="package://kuka/meshes/kr120r2500pro/visual/link_2.dae"/>
+        </geometry>
+      </visual>
+      <collision>
+        <origin xyz="0 0 0" rpy="0 0 0"/>
+        <geometry>
+          <mesh filename="package://kuka/meshes/kr120r2500pro/collision/link_2.stl" />
         </geometry>
       </collision>
@@ -73,11 +73,11 @@
         <origin xyz="0 0 0" rpy="0 0 0"/>
         <geometry>
-          <mesh filename="package://kuka_kr120_support/meshes/kr120r2500pro/visual/link_3.dae" />
-        </geometry>
-      </visual>
-      <collision>
-        <origin xyz="0 0 0" rpy="0 0 0"/>
-        <geometry>
-          <mesh filename="package://kuka_kr120_support/meshes/kr120r2500pro/collision/link_3.stl" />
+          <mesh filename="package://kuka/meshes/kr120r2500pro/visual/link_3.dae" />
+        </geometry>
+      </visual>
+      <collision>
+        <origin xyz="0 0 0" rpy="0 0 0"/>
+        <geometry>
+          <mesh filename="package://kuka/meshes/kr120r2500pro/collision/link_3.stl" />
         </geometry>
       </collision>
@@ -93,11 +93,11 @@
         <origin xyz="0 0 0" rpy="0 0 0"/>
         <geometry>
-          <mesh filename="package://kuka_kr120_support/meshes/kr120r2500pro/visual/link_4.dae" />
-        </geometry>
-      </visual>
-      <collision>
-        <origin xyz="0 0 0" rpy="0 0 0"/>
-        <geometry>
-          <mesh filename="package://kuka_kr120_support/meshes/kr120r2500pro/collision/link_4.stl" />
+          <mesh filename="package://kuka/meshes/kr120r2500pro/visual/link_4.dae" />
+        </geometry>
+      </visual>
+      <collision>
+        <origin xyz="0 0 0" rpy="0 0 0"/>
+        <geometry>
+          <mesh filename="package://kuka/meshes/kr120r2500pro/collision/link_4.stl" />
         </geometry>
       </collision>
@@ -113,11 +113,11 @@
         <origin xyz="0 0 0" rpy="0 0 0"/>
         <geometry>
-          <mesh filename="package://kuka_kr120_support/meshes/kr120r2500pro/visual/link_5.dae" />
-        </geometry>
-      </visual>
-      <collision>
-        <origin xyz="0 0 0" rpy="0 0 0"/>
-        <geometry>
-          <mesh filename="package://kuka_kr120_support/meshes/kr120r2500pro/collision/link_5.stl" />
+          <mesh filename="package://kuka/meshes/kr120r2500pro/visual/link_5.dae" />
+        </geometry>
+      </visual>
+      <collision>
+        <origin xyz="0 0 0" rpy="0 0 0"/>
+        <geometry>
+          <mesh filename="package://kuka/meshes/kr120r2500pro/collision/link_5.stl" />
         </geometry>
       </collision>
@@ -133,11 +133,11 @@
         <origin xyz="0 0 0" rpy="0 0 0"/>
         <geometry>
-          <mesh filename="package://kuka_kr120_support/meshes/kr120r2500pro/visual/link_6.dae" />
-        </geometry>
-      </visual>
-      <collision>
-        <origin xyz="0 0 0" rpy="0 0 0"/>
-        <geometry>
-          <mesh filename="package://kuka_kr120_support/meshes/kr120r2500pro/collision/link_6.stl" />
+          <mesh filename="package://kuka/meshes/kr120r2500pro/visual/link_6.dae" />
+        </geometry>
+      </visual>
+      <collision>
+        <origin xyz="0 0 0" rpy="0 0 0"/>
+        <geometry>
+          <mesh filename="package://kuka/meshes/kr120r2500pro/collision/link_6.stl" />
         </geometry>
       </collision>
@@ -219,9 +219,60 @@
         <plugin filename="libgz_ros2_control-system.so" name="gz_ros2_control::GazeboSimROS2ControlPlugin">
             <!-- <parameters>/home/hak/Desktop/synced/work/sem6/edi/jazzy_ws/install/kuka/share/kuka/config/controllers.yaml</parameters> -->
-            <ros>
+            <!-- <ros>
                <remapping>/controller_manager/robot_description:=/robot_description</remapping>
-            </ros>
+            </ros> -->
+        </plugin>
+        <plugin filename="gz-sim-joint-state-publisher-system"
+          name="gz::sim::systems::JointStatePublisher">
+          <topic>joint_states</topic> <!--from <ros><remapping> -->
+          <joint_name>joint_a1</joint_name>
+          <joint_name>joint_a2</joint_name>
+          <joint_name>joint_a3</joint_name>
+          <joint_name>joint_a4</joint_name>
+          <joint_name>joint_a5</joint_name>
+          <joint_name>joint_a6</joint_name>
+        </plugin>
+        <plugin
+          filename="gz-sim-joint-trajectory-controller-system"
+          name="gz::sim::systems::JointTrajectoryController">
+          <!-- Note: You can also specify a custom topic for the joint trajectory commands -->
+          <topic>/Arm_controller/joint_trajectory</topic>
         </plugin>
     </gazebo>
+    <ros2_control name="GazeboSimSystem" type="system">
+      <hardware>
+        <plugin>mock_components/GenericSystem</plugin>
+      </hardware>
+        <joint name="joint_a1">
+            <command_interface name="position"/>
+            <state_interface name="position"/>
+            <state_interface name="velocity"/>
+        </joint>
+        <joint name="joint_a2">
+            <command_interface name="position"/>
+            <state_interface name="position"/>
+            <state_interface name="velocity"/>
+        </joint>
+        <joint name="joint_a3">
+            <command_interface name="position"/>
+            <state_interface name="position"/>
+            <state_interface name="velocity"/>
+        </joint>
+        <joint name="joint_a4">
+            <command_interface name="position"/>
+            <state_interface name="position"/>
+            <state_interface name="velocity"/>
+        </joint>
+        <joint name="joint_a5">
+            <command_interface name="position"/>
+            <state_interface name="position"/>
+            <state_interface name="velocity"/>
+        </joint>
+        <joint name="joint_a6">
+            <command_interface name="position"/>
+            <state_interface name="position"/>
+            <state_interface name="velocity"/>
+        </joint>
+    </ros2_control>
   </xacro:macro>
 </robot>
